File: brains/brains.sch (KiCad schematic (older format))
At the start: 20 parts, among them U1 WiiChuckCon, U10 Servo, U11 Servo, U12 Servo, U13 XBEE, U2 Nokia_5510_LCD, U3 promicro, U4 JoyConnectISP, U5 JACK_2MM1, U6 TXB0108PWR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

Commit message: V1.0 Update
Kickstarter Production version
Parts:
- removed C1, C3: C, SMD_Packages:SMD-1206_Pol, symbol C
- removed D1: DIODE, SMD_Packages:SMD-1206_Pol, symbol DIODE
- removed R1: R, SMD_Packages:SMD-1206_Pol, symbol R
- removed U6: TXB0108PWR, SMD_Packages:SSOP-20, symbol TXB0108PWR
- added C4: C, Capacitors_SMD:C_0805, symbol C
- added F1, F2, F3, F4: FUSE, Brains:Surface_Mount_1812_Polyfuse, symbol FUSE
- C1: renamed from C2; footprint SMD_Packages:SMD-4032 -> Brains:EEE1CA471UP_Capacitor
- C2: renamed from C4; value C -> 10uF; footprint SMD_Packages:SMD-1206_Pol -> Capacitors_SMD:C_0805
- C3: renamed from C5; value C -> 22uF; footprint SMD_Packages:SMD-1206_Pol -> Capacitors_SMD:C_1206
- renumbered U13 to U6
Connections:
- net labels removed: +5V, 3V_BT_RX, 3V_BT_TX, 3V_LCD_CE, 3V_LCD_DC, 3V_LCD_RST, 3V_MOSI_D16, 3V_SCLK_D15
- wire segments 40 -> 30
- no-connect marks 27 -> 28
Other:
- moved on the sheet: U10, U11, U12, U9
